File: power_distribution_board_pcb_v2-2026-04-06_225556/power_distribution_board_pcb_v2.kicad_sch (KiCad schematic)
At the start: 26 parts, among them U1 LM70660RRXR

Commit message: Update KiCad project files
Parts:
- removed RFB1: 100k, symbol Device:R
- added 12V_Connector1, 3.3V_Connector1, 5V_Connector1, ESC_Connector1, ESC_Connector2, ESC_Connector3, ESC_Connector4, Tether_Connector1: Conn_01x02, TerminalBlock_Phoenix:TerminalBlock_Phoenix_MKDS-1,5-2-5.08_1x02_P5.08mm_Horizontal, symbol Connector_Generic:Conn_01x02
- added C1: 2.2nF, Capacitor_SMD:C_0805_2012Metric_Pad1.18x1.45mm_HandSolder, symbol Device:C
- added CBOOT2, CVCC2: 4.7, Capacitor_SMD:C_0805_2012Metric_Pad1.18x1.45mm_HandSolder, symbol Device:C
- added CCOMP2: 10nF, Capacitor_SMD:C_0805_2012Metric_Pad1.18x1.45mm_HandSolder, symbol Device:C
- added CF1, CF2: 22uF, Capacitor_SMD:C_1210_3225Metric_Pad1.33x2.70mm_HandSolder, symbol Device:C
- added CHF2: 150pF, Capacitor_SMD:C_0805_2012Metric_Pad1.18x1.45mm_HandSolder, symbol Device:C
- added CIN10, CIN9: 10uF, Capacitor_SMD:C_0805_2012Metric_Pad1.18x1.45mm_HandSolder, symbol Device:C
- added CIN5, CIN6, CIN7, CIN8: 4.7µF, Capacitor_SMD:C_1210_3225Metric_Pad1.33x2.70mm_HandSolder, symbol Device:C
- added COUT10, COUT11, COUT9: 22uF, Capacitor_SMD:C_0805_2012Metric_Pad1.18x1.45mm_HandSolder, symbol Device:C
- added COUT5, COUT6, COUT7, COUT8: 47, Capacitor_SMD:C_1210_3225Metric_Pad1.33x2.70mm_HandSolder, symbol Device:C
- added CVDDA2: 0.1, Capacitor_SMD:C_0805_2012Metric_Pad1.18x1.45mm_HandSolder, symbol Device:C
- added C_IN-HF2: 0.1 µF, Capacitor_SMD:C_0805_2012Metric_Pad1.18x1.45mm_HandSolder, symbol Device:C
- added C_NR/SS1: 470nF, Capacitor_SMD:C_0805_2012Metric_Pad1.18x1.45mm_HandSolder, symbol Device:C
- added FB1: FerriteBead, Inductor_SMD:L_0603_1608Metric_Pad1.05x0.95mm_HandSolder, symbol Device:FerriteBead
- added L1: 2.2uH, Coilcraft:IND_XGL4030_COC-M, symbol Device:L
- added Lo2: 3.3, Coilcraft:IND_XGL4030_COC-M, symbol Device:L
- added R3, R6, REN4: 100k, Resistor_SMD:R_0805_2012Metric_Pad1.20x1.40mm_HandSolder, symbol Device:R
- added R4: 31.6k, Resistor_SMD:R_0805_2012Metric_Pad1.20x1.40mm_HandSolder, symbol Device:R
- added R5: 52.3k, Resistor_SMD:R_0805_2012Metric_Pad1.20x1.40mm_HandSolder, symbol Device:R
- added R7: 4.87k, Resistor_SMD:R_0805_2012Metric_Pad1.20x1.40mm_HandSolder, symbol Device:R
- added R8: 2.49k, Resistor_SMD:R_0805_2012Metric_Pad1.20x1.40mm_HandSolder, symbol Device:R
- added RBOOT2: 1Ohm, Resistor_SMD:R_0805_2012Metric_Pad1.20x1.40mm_HandSolder, symbol Device:R
- added RCNFG2: 29.4K, Resistor_SMD:R_0805_2012Metric_Pad1.20x1.40mm_HandSolder, symbol Device:R
- added RCOMP2: 3.24k, Resistor_SMD:R_0805_2012Metric_Pad1.20x1.40mm_HandSolder, symbol Device:R
- added REN3: 20.5k, Resistor_SMD:R_0805_2012Metric_Pad1.20x1.40mm_HandSolder, symbol Device:R
- added RRT2: R, Resistor_SMD:R_0805_2012Metric_Pad1.20x1.40mm_HandSolder, symbol Device:R
- added RS2: 5m, Resistor_SMD:R_0805_2012Metric_Pad1.20x1.40mm_HandSolder, symbol Device:R
- added U2: LM70660RRXR, Lm70660:RRX0029B-MFG, symbol Lm70660:LM70660RRXR
- added U3: TPS62913, Package_DFN_QFN:Texas_RPU0010A_VQFN-HR-10_2x2mm_P0.5mm, symbol Regulator_Switching:TPS62913
- CBOOT1: renamed from CBOOT; value 4.7 -> 47nF; footprint (none) -> Capacitor_SMD:C_0805_2012Metric_Pad1.18x1.45mm_HandSolder
- CCOMP1: renamed from CCOMP; value 6.8 -> 10nF; footprint (none) -> Capacitor_SMD:C_0805_2012Metric_Pad1.18x1.45mm_HandSolder
- CHF1: renamed from CHF; value 47 -> 150pF; footprint (none) -> Capacitor_SMD:C_0805_2012Metric_Pad1.18x1.45mm_HandSolder
- CIN1, CIN2, CIN3, CIN4: footprint (none) -> Capacitor_SMD:C_1210_3225Metric_Pad1.33x2.70mm_HandSolder
- COUT1, COUT2, COUT3, COUT4: value 47 -> 47uF; footprint (none) -> Capacitor_SMD:C_1210_3225Metric_Pad1.33x2.70mm_HandSolder
- CVCC1: renamed from CVCC; value 4.7 -> 4.7uF; footprint (none) -> Capacitor_SMD:C_0805_2012Metric_Pad1.18x1.45mm_HandSolder
- CVDDA1: renamed from CVDDA; value 0.1 -> 0.1uF; footprint (none) -> Capacitor_SMD:C_0805_2012Metric_Pad1.18x1.45mm_HandSolder
- C_IN-HF1: renamed from C_IN-HF; footprint (none) -> Capacitor_SMD:C_0805_2012Metric_Pad1.18x1.45mm_HandSolder
- Lo1: renamed from Lo; value 3.3 -> 2.2uH; footprint (none) -> Coilcraft:IND_XGL4030_COC-M
- R1: value 100 -> 100kF; footprint (none) -> Resistor_SMD:R_0805_2012Metric_Pad1.20x1.40mm_HandSolder
- R2: value 19.1 -> 31.6kF; footprint (none) -> Resistor_SMD:R_0805_2012Metric_Pad1.20x1.40mm_HandSolder
- RBOOT1: renamed from RBOOT; footprint (none) -> Resistor_SMD:R_0805_2012Metric_Pad1.20x1.40mm_HandSolder
- RCNFG1: renamed from RCNFG; footprint (none) -> Resistor_SMD:R_0805_2012Metric_Pad1.20x1.40mm_HandSolder
- RCOMP1: renamed from RCOMP; value 5.76 -> 3.24kF; footprint (none) -> Resistor_SMD:R_0805_2012Metric_Pad1.20x1.40mm_HandSolder
- REN1, REN2: footprint (none) -> Resistor_SMD:R_0805_2012Metric_Pad1.20x1.40mm_HandSolder
- RRT1: renamed from RRT; value R -> 54.9K; footprint (none) -> Resistor_SMD:R_0805_2012Metric_Pad1.20x1.40mm_HandSolder
- RS1: renamed from RS; value 5m -> 4mQ; footprint (none) -> Resistor_SMD:R_0805_2012Metric_Pad1.20x1.40mm_HandSolder
Connections:
- net EN_VULO is gone; now on net EN_UVLO_12V: REN1.1
- net +48V: now also CIN5.1, CIN6.2, CIN7.2, CIN8.2, C_IN-HF2.1, ESC_Connector1.1 (Pin_1), ESC_Connector2.1 (Pin_1), ESC_Connector3.1 (Pin_1), ESC_Connector4.1 (Pin_1), REN3.2, REN4.2, Tether_Connector1.1 (Pin_1), U2.1 (VIN4), U2.2 (VIN5), U2.27 (VIN1), U2.28 (VIN2), U2.29 (VIN3), U2.3 (VIN6)
- net CONFIG: now also RCNFG2.1, U2.13 (CONFIG); no longer RCNFG1.1
- net EXTCOMP: now also CHF2.2, RCOMP2.2, U2.15 (EXTCOMP); no longer CHF1.2, RCOMP1.2
- net RT: now also RRT2.1, U2.14 (RT); no longer RRT1.1
- net VDDA: now also CVDDA2.1, U2.18 (VDDA); no longer CVDDA1.1
- net GND: now reaches CCOMP1.1, CHF1.1, CIN1.1, CIN2.1, CIN3.2, CIN4.1, COUT1.2, COUT2.2, COUT3.2, COUT4.2, CVCC1.2, CVDDA1.2, C_IN-HF1.2, R2.2, RCNFG1.2, REN2.1, RRT1.2, U1.17 (AGND), U1.23 (PGND1), U1.24 (PGND2), U1.25 (PGND3), U1.26 (PGND4), U1.30 (PGND), U1.8 (PFM_SYNCIN)
- net GND: now also 12V_Connector1.2 (Pin_2), 3.3V_Connector1.2 (Pin_2), 5V_Connector1.2 (Pin_2), C1.2, CCOMP2.1, CF2.2, CHF2.1, CIN10.2, CIN5.2, CIN6.1, CIN7.1, CIN8.1, COUT11.2, COUT5.2, COUT6.2, COUT7.2, COUT8.2, CVCC2.2, C_IN-HF2.2, C_NR/SS1.1, ESC_Connector1.2 (Pin_2), ESC_Connector2.2 (Pin_2), ESC_Connector3.2 (Pin_2), ESC_Connector4.2 (Pin_2), R4.2, R5.2, R7.2, REN3.1, Tether_Connector1.2 (Pin_2), U2.17 (AGND), U2.23 (PGND1), U2.24 (PGND2), U2.25 (PGND3), U2.26 (PGND4), U2.30 (PGND), U2.8 (PFM_SYNCIN), U3.4 (PGND), U3.7 (PSNS); no longer COUT1.1, COUT2.1, COUT3.1, COUT4.1, R1.1, RS1.2, U1.12 (VOUT), U1.6 (BIAS)
- net FB_12V: now reaches R1.2, R2.1
- net FB_12V: now also U1.16 (FB)
- net CONFIG_12V: now reaches U1.13 (CONFIG)
- net CONFIG_12V: now also RCNFG1.1
- net RT_12V: now reaches U1.14 (RT)
- net RT_12V: now also RRT1.1
- net EXTCOMP_12V: now reaches U1.15 (EXTCOMP)
- net EXTCOMP_12V: now also CHF1.2, RCOMP1.2
- net VDDA_12V: now reaches U1.18 (VDDA)
- net VDDA_12V: now also CVDDA1.1
- net EN_UVLO_12V: now reaches U1.9 (EN_UVLO)
- new net: CBOOT2.1, U2.4 (CBOOT)
- new net: CBOOT2.2, RBOOT2.1, U2.20 (SW1), U2.21 (SW2), U2.22 (SW3), U2.5 (SW4)
- new net: CIN10.1, CIN9.2
- new net: CF1.2, CF2.1
- new net: COUT10.1, COUT9.2
- new net: COUT10.2, COUT11.1
- new net: R7.1, R8.2, U3.9 (FB)
- new net: Lo2.1, RBOOT2.2
- new net: Lo2.2, RS2.1, U2.11 (ISNS+)
- new net: R6.1, U3.5 (PG)
- new net: R5.1, U3.10 (S-CONF)
- new net: L1.1, U3.2 (SW)
- new net: COUT9.1, FB1.1, L1.2, U3.3 (VO)
- new net: CCOMP2.2, RCOMP2.1
- new net: CVCC2.1, U2.19 (VCC)
- new net 12V_BUS: 12V_Connector1.1 (Pin_1), COUT1.1, COUT2.1, COUT3.1, COUT4.1, R1.1, RS1.2, U1.12 (VOUT), U1.6 (BIAS)
- new net 3.3V_BUS: 3.3V_Connector1.1 (Pin_1), CF1.1, FB1.2, R6.2, R8.1
- new net 5V_BUS: 5V_Connector1.1 (Pin_1), C1.1, CIN9.1, COUT5.1, COUT6.1, COUT7.1, COUT8.1, R3.1, RS2.2, U2.12 (VOUT), U2.6 (BIAS), U3.1 (EN/SYNC), U3.6 (VIN)
- new net AGND: CVDDA2.2, RCNFG2.2, RRT2.2
- new net EN_UVLO: REN4.1, U2.9 (EN_UVLO)
- new net FB_5V: R3.2, R4.1, U2.16 (FB)
- new net NR/SS: C_NR/SS1.2, U3.8 (NR/SS)
- no-connect marks 0 -> 4
Other:
- moved on the sheet: CBOOT1, CCOMP1, CHF1, CIN1, CIN3, CIN4, COUT1, COUT2, COUT3, COUT4, CVCC1, CVDDA1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
