File: power_distribution_board_pcb_v2-2026-04-06_225556/power_distribution_board_pcb_v2.kicad_pcb (KiCad board)
At the start: 2 copper layers, 126 x 53.4 mm, 78 parts, among them U1 LM70660RRXR, U2 LM70660RRXR, U3 TPS62913

Commit message: update pcb and schematic
Routing:
- net GND: track 83.5 -> 552.2 mm, vias 37 -> 172
- net /3.3V_BUS: track 54.1 -> 55.8 mm
- net Net-(U3-PG): track 3.03 -> 4.13 mm
