File: power_distribution_board_pcb_v2-2026-04-06_225556/power_distribution_board_pcb_v2.kicad_pcb (KiCad board)
At the start: 2 copper layers, 126 x 53.4 mm, 78 parts, among them U1 LM70660RRXR, U2 LM70660RRXR, U3 TPS62913

Commit message: Add power distribution board files
Routing:
- net /12V_BUS: track 152.1 -> 149.6 mm
- net Net-(Lo2-Pad1): vias 0 -> 1
- added copper zone on F.Cu, net GND
Changed lines of the file:
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@@
 			(pinfunction "PGND_30")
 			(pintype "power_in")
+			(zone_connect 2)
 		)
 		(pad "31" thru_hole circle
@@
 			(remove_unused_layers no)
 			(net "GND")
+			(zone_connect 2)
 		)
 		(pad "36" thru_hole circle
@@
 			(remove_unused_layers no)
 			(net "GND")
+			(zone_connect 2)
 		)
 		(pad "37" thru_hole circle
@@
 			(remove_unused_layers no)
 			(net "GND")
+			(zone_connect 2)
 		)
 		(pad "32" thru_hole circle
@@
 			(remove_unused_layers no)
 			(net "GND")
+			(zone_connect 2)
 		)
 		(pad "33" thru_hole circle
@@
 			(remove_unused_layers no)
 			(net "GND")
+			(zone_connect 2)
 		)
 		(pad "34" thru_hole circle
@@
 			(remove_unused_layers no)
 			(net "GND")
+			(zone_connect 2)
 		)
 		(pad "35" thru_hole circle
@@
 			(remove_unused_layers no)
 			(net "GND")
+			(zone_connect 2)
 		)
 		(pad "36" thru_hole circle
@@
 			(remove_unused_layers no)
 			(net "GND")
+			(zone_connect 2)
 		)
 		(pad "37" thru_hole circle
@@
 	)
 	(segment
-		(start 186.8675 91.9525)
-		(end 185.42 93.4)
-		(width 0.5)
-		(layer "F.Cu")
-		(net "/12V_BUS")
-	)
-	(segment
 		(start 189.134999 91.61)
 		(end 188.84 91.61)
@@
 	)
 	(segment
-		(start 186.8675 91.46)
-		(end 186.8675 91.9525)
-		(width 0.5)
-		(layer "F.Cu")
-		(net "/12V_BUS")
-	)
-	(segment
 		(start 114.6988 111.86)
 		(end 118.7188 115.88)
@@
 		(net "Net-(Lo2-Pad1)")
 	)
+	(via
+		(at 148.38 100.96)
+		(size 0.6)
+		(drill 0.3)
+		(layers "F.Cu" "B.Cu")
+		(net "Net-(Lo2-Pad1)")
+	)
 	(segment
 		(start 194.865 97.26)
@@
 	(zone
 		(net "GND")
-		(layer "B.Cu")
+		(layers "F.Cu" "B.Cu")
 		(hatch edge 0.5)
-		(connect_pads yes
+		(connect_pads
 			(clearance 0.5)
 		)
